Commit message: Update default URDF to A1Z_Flange and sync inertial params to A1Z_G1Z
- Default URDF changed from A1Z_2kg to A1Z_Flange (bare flange, no payload)
- README: update examples, remove nogripper/2kg references, fix gravity
  sign description (joint3 reversed, not joint4)
- A1Z_G1Z.urdf: sync arm_link3/4 calibrated inertial properties from
  A1Z_Flange (mass, CoM, inertia tensor)

Co-Authored-By: Claude Opus 4.6 (1M context) <noreply@anthropic.com>

File: a1z/robot_models/a1z/A1Z_G1Z.urdf (robot description, URDF)
Before this commit: robot A1Z_G1Z, 9 links, 8 joints
Links:
- link arm_link3: mass 0.93954481 -> 0.99109270
- link arm_link4: mass 0.17709874 -> 0.48309874
