Commit message: Unify joint coordinate system and fix J3 limits
- Add joint_sign at motor I/O boundary so all state/commands use URDF frame
- Remove gravity_torque_sign from torque computation (replaced by joint_sign)
- Fix J3 joint limits to (-3.142, 0.0) matching URDF frame
- Fix A1Z_Flange.urdf J3 limit to lower=-3.142, upper=0
- Update README control formula and parameter descriptions

File: a1z/robot_models/a1z/A1Z_Flange.urdf (robot description, URDF)
Before this commit: robot A1Z_Flange, 7 links, 6 joints
Joints:
- joint arm_joint3: limit lower=0 upper=3.142 effort=0 velocity=0 -> lower=-3.142 upper=0 effort=0 velocity=0

Commit message: update A1Z_Flange.urdf

File: a1z/robot_models/a1z/A1Z_Flange.urdf (robot description, URDF)
Before this commit: robot A1Z_Flange, 7 links, 6 joints
Joints:
- joint arm_joint1: limit lower=-2.094 upper=2.094 effort=0 velocity=0 -> lower=-2.094 upper=2.094 effort=20 velocity=5.65
- joint arm_joint2: limit lower=0 upper=3.142 effort=0 velocity=0 -> lower=0 upper=3.142 effort=25 velocity=5.65
- joint arm_joint3: limit lower=-3.142 upper=0 effort=0 velocity=0 -> lower=-3.142 upper=0 effort=20 velocity=5.65
- joint arm_joint4: limit lower=-1.309 upper=1.309 effort=0 velocity=0 -> lower=-1.309 upper=1.309 effort=9 velocity=3.77
- joint arm_joint5: limit lower=-1.484 upper=1.484 effort=0 velocity=0 -> lower=-1.484 upper=1.484 effort=3.5 velocity=10.47
- joint arm_joint6: limit lower=-2.007 upper=2.007 effort=0 velocity=0 -> lower=-2.007 upper=2.007 effort=3.5 velocity=10.47
