Commit message: feat: 以本地 SDK 为准同步（优化/标定/看门狗工具与测试）
- analysis: 新增 optimize/ 模块与 optimize.sh、verify.sh
- analysis/script: 新增 a2/a3 gate 评估、看门狗标定、cost v4 重算、优化运行、结果校验脚本
- robots: 调整 arm_robot/get_robot/integrator 实现
- tests: 新增 cost_spec、friction、merge_gains、search_space、vel_ff、warm_start、watchdog 测试

File: a1z/robot_models/a1z/A1Z_Flange.urdf (robot description, URDF)
Before this commit: robot A1Z_Flange, 7 links, 6 joints
Joints:
- joint arm_joint2: limit lower=0 upper=3.142 effort=25 velocity=5.65 -> lower=-3.142 upper=3.142 effort=25 velocity=5.65

File: a1z/robot_models/a1z/A1Z_G1Z.urdf (robot description, URDF)
Before this commit: robot A1Z_G1Z, 9 links, 8 joints
Joints:
- joint arm_joint2: limit lower=0 upper=3.142 effort=25 velocity=5.65 -> lower=-3.142 upper=3.142 effort=25 velocity=5.65

Commit message: feat: 更新库仑摩擦扭矩先 验估计

File: a1z/robot_models/a1z/A1Z_Flange.urdf (robot description, URDF)
Before this commit: robot A1Z_Flange, 7 links, 6 joints
Joints:
- joint arm_joint2: limit lower=-3.142 upper=3.142 effort=25 velocity=5.65 -> lower=0 upper=3.142 effort=25 velocity=5.65

File: a1z/robot_models/a1z/A1Z_G1Z.urdf (robot description, URDF)
Before this commit: robot A1Z_G1Z, 9 links, 8 joints
Joints:
- joint arm_joint2: limit lower=-3.142 upper=3.142 effort=25 velocity=5.65 -> lower=0 upper=3.142 effort=25 velocity=5.65
